File: hardware/yardforce/MowerConnectors.kicad_sch (KiCad schematic)
At the start: 12 parts, among them J3 YF-Rev6-B, J4 YF-Rev4-A, J5 YF-Rev6-A, J6 YF-Rev4-B, J7 OM UI Board, J8 Shell Stop, J9 Rain

Commit message: Prepared HW v0.3
Parts:
- JP1, JP2: footprint Jumper:SolderJumper-2_P1.3mm_Open_RoundedPad1.0x1.5mm -> Jumper:SolderJumper-2_P1.3mm_Bridged_RoundedPad1.0x1.5mm; symbol Jumper:SolderJumper_2_Open -> Jumper:SolderJumper_2_Bridged
Connections:
- net RAIN_OEM: now reaches J3.11 (Pin_11)
- net RAIN_OEM: now also J5.11 (Pin_11)
- net BTN_ANY: now reaches J3.2 (Pin_2)
- net BTN_ANY: now also J5.2 (Pin_2)
- no-connect marks 22 -> 18
Other:
- note removed: "BTN_ANY"
Changed lines of the file:
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@@
 	)
 	(no_connect
-		(at 167.64 57.15)
-	)
-	(no_connect
 		(at 100.33 93.98)
 	)
@@
 	)
 	(no_connect
-		(at 100.33 44.45)
-	)
-	(no_connect
 		(at 100.33 121.92)
 	)
@@
 	)
 	(no_connect
-		(at 87.63 57.15)
-	)
-	(no_connect
-		(at 180.34 44.45)
-	)
-	(no_connect
 		(at 100.33 119.38)
 	)
@@
 	(wire
 		(pts
+			(xy 82.55 49.53) (xy 87.63 49.53)
+		)
+		(stroke
+			(width 0)
+			(type default)
+		)
+	)
+	(wire
+		(pts
 			(xy 180.34 127) (xy 195.58 127)
 		)
@@
 	(wire
 		(pts
-			(xy 162.56 54.61) (xy 167.64 54.61)
+			(xy 149.86 54.61) (xy 167.64 54.61)
 		)
 		(stroke
@@
 	(wire
 		(pts
-			(xy 154.94 44.45) (xy 167.64 44.45)
+			(xy 149.86 44.45) (xy 167.64 44.45)
 		)
 		(stroke
@@
 	(wire
 		(pts
+			(xy 100.33 44.45) (xy 114.3 44.45)
+		)
+		(stroke
+			(width 0)
+			(type default)
+		)
+	)
+	(wire
+		(pts
+			(xy 162.56 49.53) (xy 167.64 49.53)
+		)
+		(stroke
+			(width 0)
+			(type default)
+		)
+	)
+	(wire
+		(pts
 			(xy 167.64 119.38) (xy 154.94 119.38)
 		)
@@
 	(wire
 		(pts
-			(xy 82.55 54.61) (xy 87.63 54.61)
+			(xy 72.39 54.61) (xy 87.63 54.61)
 		)
 		(stroke
@@
 	(wire
 		(pts
-			(xy 83.82 62.23) (xy 87.63 62.23)
+			(xy 82.55 62.23) (xy 87.63 62.23)
 		)
 		(stroke
@@
 	(wire
 		(pts
-			(xy 74.93 46.99) (xy 87.63 46.99)
+			(xy 69.85 46.99) (xy 87.63 46.99)
 		)
 		(stroke
@@
 	(wire
 		(pts
+			(xy 162.56 57.15) (xy 167.64 57.15)
+		)
+		(stroke
+			(width 0)
+			(type default)
+		)
+	)
+	(wire
+		(pts
 			(xy 180.34 99.06) (xy 196.85 99.06)
 		)
@@
 	(wire
 		(pts
-			(xy 154.94 46.99) (xy 167.64 46.99)
+			(xy 149.86 46.99) (xy 167.64 46.99)
 		)
 		(stroke
@@
 	(wire
 		(pts
+			(xy 69.85 57.15) (xy 87.63 57.15)
+		)
+		(stroke
+			(width 0)
+			(type default)
+		)
+	)
+	(wire
+		(pts
 			(xy 118.11 176.53) (xy 120.65 176.53)
 		)
@@
 	(wire
 		(pts
-			(xy 74.93 44.45) (xy 87.63 44.45)
+			(xy 69.85 44.45) (xy 87.63 44.45)
 		)
 		(stroke
@@
 	(wire
 		(pts
-			(xy 163.83 62.23) (xy 167.64 62.23)
+			(xy 162.56 62.23) (xy 167.64 62.23)
 		)
 		(stroke
@@
 		)
 	)
-	(text "BTN_ANY"
-		(exclude_from_sim no)
-		(at 180.594 43.688 0)
-		(effects
-			(font
-				(size 1.27 1.27)
-			)
-			(justify left)
-		)
-	)
 	(text "JP3.06?"
 		(exclude_from_sim no)
@@
 		)
 	)
-	(text "BTN_ANY"
-		(exclude_from_sim no)
-		(at 100.584 43.688 0)
-		(effects
-			(font
-				(size 1.27 1.27)
-			)
-			(justify left)
-		)
-	)
 	(text "Either use YF-Rev4-A/B or YF-Rev6-A/B connector pair.\nAdapter get get plugged to the matching CoverUI- A or B side.\nOther side get plugged either to YF-Mainboard,\nor remains free and get connected via \"OM UI Board\" plug to an OpenMower-Mainboard.\n"
 		(exclude_from_sim no)
@@
 	)
 	(label "HALL_RBUMP"
-		(at 163.83 62.23 180)
+		(at 162.56 62.23 180)
 		(fields_autoplaced yes)
 		(effects
@@
 		)
 	)
+	(label "BTN_ANY"
+		(at 180.34 44.45 0)
+		(fields_autoplaced yes)
+		(effects
+			(font
+				(size 1.27 1.27)
+			)
+			(justify left bottom)
+		)
+	)
 	(label "HALL_LBUMP"
 		(at 180.34 134.62 0)
@@
 		)
 	)
+	(label "RAIN_OEM"
+		(at 82.55 57.15 180)
+		(fields_autoplaced yes)
+		(effects
+			(font
+				(size 1.27 1.27)
+			)
+			(justify right bottom)
+		)
+	)
 	(label "BTN_PLAY"
 		(at 180.34 46.99 0)
@@
 		)
 	)
+	(label "RAIN_OEM"
+		(at 162.56 57.15 180)
+		(fields_autoplaced yes)
+		(effects
+			(font
+				(size 1.27 1.27)
+			)
+			(justify right bottom)
+		)
+	)
 	(label "HALL_LIFT"
 		(at 100.33 62.23 0)
@@
 	)
 	(label "BTN_HOME"
-		(at 87.63 49.53 180)
+		(at 82.55 49.53 180)
 		(fields_autoplaced yes)
 		(effects
@@
 	)
 	(label "BTN_HOME"
-		(at 167.64 49.53 180)
+		(at 162.56 49.53 180)
 		(fields_autoplaced yes)
 		(effects
@@
 	)
 	(label "HALL_RBUMP"
-		(at 83.82 62.23 180)
+		(at 82.55 62.23 180)
 		(fields_autoplaced yes)
 		(effects
@@
 		)
 	)
+	(label "BTN_ANY"
+		(at 100.33 44.45 0)
+		(fields_autoplaced yes)
+		(effects
+			(font
+				(size 1.27 1.27)
+			)
+			(justify left bottom)
+		)
+	)
 	(label "HALL_RBUMP"
 		(at 167.64 139.7 180)
@@
 		)
 	)
+	(hierarchical_label "BTN_ANY"
+		(shape bidirectional)
+		(at 114.3 44.45 0)
+		(fields_autoplaced yes)
+		(effects
+			(font
+				(size 1.27 1.27)
+			)
+			(justify left)
+		)
+	)
 	(hierarchical_label "LED_34HR"
 		(shape bidirectional)
@@
 	(hierarchical_label "R6A_TXD1"
 		(shape output)
-		(at 74.93 46.99 180)
+		(at 69.85 46.99 180)
 		(fields_autoplaced yes)
 		(effects
@@
 	)
 	(hierarchical_label "RAIN_SENSOR"
-		(shape output)
+		(shape bidirectional)
 		(at 118.11 176.53 180)
 		(fields_autoplaced yes)
@@
 		)
 	)
+	(hierarchical_label "RAIN_OEM"
+		(shape bidirectional)
+		(at 69.85 57.15 180)
+		(fields_autoplaced yes)
+		(effects
+			(font
+				(size 1.27 1.27)
+			)
+			(justify right)
+		)
+	)
 	(hierarchical_label "R6B_TXDX"
 		(shape output)
-		(at 154.94 46.99 180)
+		(at 149.86 46.99 180)
 		(fields_autoplaced yes)
 		(effects
@@
 	(hierarchical_label "R6B_RXDX"
 		(shape input)
-		(at 154.94 44.45 180)
+		(at 149.86 44.45 180)
 		(fields_autoplaced yes)
 		(effects
@@
 	(hierarchical_label "R6A_RXD1"
 		(shape input)
-		(at 74.93 44.45 180)
+		(at 69.85 44.45 180)
 		(fields_autoplaced yes)
 		(effects
@@
 	)
 	(symbol
-		(lib_id "Jumper:SolderJumper_2_Open")
+		(lib_id "Jumper:SolderJumper_2_Bridged")
 		(at 113.03 91.44 0)
 		(unit 1)
@@
 			)
 		)
-		(property "Footprint" "Jumper:SolderJumper-2_P1.3mm_Open_RoundedPad1.0x1.5mm"
+		(property "Footprint" "Jumper:SolderJumper-2_P1.3mm_Bridged_RoundedPad1.0x1.5mm"
 			(at 113.03 91.44 0)
 			(effects
@@
 			)
 		)
-		(property "Description" "Solder Jumper, 2-pole, open"
+		(property "Description" "Solder Jumper, 2-pole, closed/bridged"
 			(at 113.03 91.44 0)
 			(effects
@@
 	)
 	(symbol
-		(lib_id "Jumper:SolderJumper_2_Open")
+		(lib_id "Jumper:SolderJumper_2_Bridged")
 		(at 193.04 91.44 0)
 		(unit 1)
@@
 			)
 		)
-		(property "Footprint" "Jumper:SolderJumper-2_P1.3mm_Open_RoundedPad1.0x1.5mm"
+		(property "Footprint" "Jumper:SolderJumper-2_P1.3mm_Bridged_RoundedPad1.0x1.5mm"
 			(at 193.04 91.44 0)
 			(effects
@@
 			)
 		)
-		(property "Description" "Solder Jumper, 2-pole, open"
+		(property "Description" "Solder Jumper, 2-pole, closed/bridged"
 			(at 193.04 91.44 0)
 			(effects
@@
 		(lib_name "+5V_3")
 		(lib_id "power:+5V")
-		(at 82.55 54.61 90)
+		(at 72.39 54.61 90)
 		(unit 1)
 		(exclude_from_sim no)
@@
 		(dnp no)
 		(property "Reference" "#PWR019"
-			(at 86.36 54.61 0)
+			(at 76.2 54.61 0)
 			(effects
 				(font
@@
 		)
 		(property "Value" "+5V"
-			(at 77.216 54.61 90)
+			(at 67.056 54.61 90)
 			(effects
 				(font
@@
 		)
 		(property "Footprint" ""
-			(at 82.55 54.61 0)
+			(at 72.39 54.61 0)
 			(effects
 				(font
@@
 		)
 		(property "Datasheet" ""
-			(at 82.55 54.61 0)
+			(at 72.39 54.61 0)
 			(effects
 				(font
@@
 		)
 		(property "Description" "Power symbol creates a global label with name \"+5V\""
-			(at 82.55 54.61 0)
+			(at 72.39 54.61 0)
 			(effects
 				(font
@@
 		(lib_name "+5V_6")
 		(lib_id "power:+5V")
-		(at 162.56 54.61 90)
+		(at 149.86 54.61 90)
 		(unit 1)
 		(exclude_from_sim no)
@@
 		(dnp no)
 		(property "Reference" "#PWR08"
-			(at 166.37 54.61 0)
+			(at 153.67 54.61 0)
 			(effects
 				(font
@@
 		)
 		(property "Value" "+5V"
-			(at 157.226 54.61 90)
+			(at 144.526 54.61 90)
 			(effects
 				(font
@@
 		)
 		(property "Footprint" ""
-			(at 162.56 54.61 0)
+			(at 149.86 54.61 0)
 			(effects
 				(font
@@
 		)
 		(property "Datasheet" ""
-			(at 162.56 54.61 0)
+			(at 149.86 54.61 0)
 			(effects
 				(font
@@
 		)
 		(property "Description" "Power symbol creates a global label with name \"+5V\""
-			(at 162.56 54.61 0)
+			(at 149.86 54.61 0)
 			(effects
 				(font
