File: hardware/yardforce/YF-Rev4-6-Adapter.kicad_sch (KiCad schematic)
At the start: 55 parts, among them J1 USB_OTG, J2 TC2050-IDC, J3 YF-Rev6-B, J4 YF-Rev6-A, J5 YF-Rev4-A, J6 YF-Rev4-B, J7 OM UI Board, J8 Shell Stop, J9 Rain, U1 AMS1117-3.3, U3 TCA9555PWR, U4 ESP32-S3-FH4R2, Y1 40MHz 10.5pF ±10ppm

Commit message: Rev 0.2 hardware
Parts:
- removed C4: .1uF, Capacitor_SMD:C_0402_1005Metric, symbol Device:C
- removed D4: PDZ3.3B,115, Diode_SMD:D_SOD-323, symbol Device:D_Zener
- removed J3: YF-Rev6-B, libs:IDC-Hybrid_2x08_P2.54mm_Latch_Vertical, symbol Connector_Generic:Conn_02x08_Odd_Even
- removed J4: YF-Rev6-A, libs:IDC-Hybrid_2x08_P2.54mm_Latch_Vertical, symbol Connector_Generic:Conn_02x08_Odd_Even
- removed J5: YF-Rev4-A, libs:IDC-Hybrid_2x20_P2.54mm_Latch_Vertical, symbol Connector_Generic:Conn_02x20_Odd_Even
- removed J6: YF-Rev4-B, libs:IDC-Hybrid_2x20_P2.54mm_Latch_Vertical, symbol Connector_Generic:Conn_02x20_Odd_Even
- removed J7: OM UI Board, Connector_JST:JST_XH_B4B-XH-A_1x04_P2.50mm_Vertical, symbol Connector_Generic:Conn_01x04
- removed J8: Shell Stop, Connector_JST:JST_XH_B3B-XH-A_1x03_P2.50mm_Vertical, symbol Connector_Generic:Conn_01x03
- removed J9: Rain, Connector_JST:JST_XH_B2B-XH-A_1x02_P2.50mm_Vertical, symbol Connector_Generic:Conn_01x02
- removed JP2: Rev4-A 3.3V, Jumper:SolderJumper-2_P1.3mm_Open_RoundedPad1.0x1.5mm, symbol Jumper:SolderJumper_2_Open
- removed JP3: Rev4-B 3.3V, Jumper:SolderJumper-2_P1.3mm_Open_RoundedPad1.0x1.5mm, symbol Jumper:SolderJumper_2_Open
- removed R12: 10k, Resistor_SMD:R_0603_1608Metric, symbol Device:R
- added C13, C5: .1uF, Capacitor_SMD:C_0402_1005Metric, symbol Device:C
- added D5: D_Schottky, Diode_SMD:D_SOD-123, symbol Device:D_Schottky
- added D6, D7, D8, D9: D_TVS, Diode_SMD:D_SOD-523, symbol Device:D_TVS
- added J10: IPEX/U.FL, libs:IPEX-SMD_BWIPX-1-001E, symbol 20279-001E-03:20279-001E-03
- added R13: 10k, Resistor_SMD:R_0603_1608Metric, symbol Device:R
- added R14, R15: 0, Resistor_SMD:R_0402_1005Metric, symbol Device:R
- C1: value 10uF -> 22uF; footprint Capacitor_SMD:C_0603_1608Metric -> Capacitor_SMD:C_0805_2012Metric; LCSC C19702 -> C45783; Stock_PN C-0603-10uF-10V -> CL21A226MAQNNNE
- C2: value 10uF -> 22uF/10V; footprint Capacitor_SMD:C_0603_1608Metric -> libs:CASE-A_3216; symbol Device:C -> CASE-A_3216:CA45-A-10V-22UF-K; LCSC C19702 -> C129272; Stock_PN C-0603-10uF-10V -> CA45-A-10V-22uF-K Copy
- D1: Digikey 1727-5192-1-ND -> (none); LCSC C82288 -> C82544; Part Number PMEG2010ER,115 -> 1N5819HW-7-F; Stock_PN D-PMEG2010ER -> 1N5819HW-7-F
- J2: now left out of the parts list
- R3, R4, R5: value 22 -> 470; LCSC C23345 -> C23179
- R8: value 200 -> 220; LCSC C8218 -> C22962
Connections:
- net BTN_10H/R3 is gone; now on net BTN_S1: U3.19 (P16)
- net BTN_6H/R5 is gone; now on net BTN_LOCK: U3.17 (P14)
- net BTN_8H/ADS7843_PEN_IRQ is gone; now on net BTN_S2: U3.18 (P15)
- net LED_10H/LCD is gone; now on net LCD_BACKLIGHT: U4.18 (GPIO13/ADC2_CH2)
- net LED_4H/LCD is gone; now on net LED_LOCK: U4.15 (GPIO10/ADC1_CH9)
- net LED_8H/R1 is gone; now on net LED_S2: U4.17 (GPIO12/ADC2_CH1)
- net LED_BAT_ADS7843-DOUT is gone; now on net BTN_HOME: U4.8 (GPIO3/ADC1_CH2)
- net +3V3: now also C13.1, R13.2
- net +5V: now also C5.1, D5.1 (K)
- net BTN_HOME: now also R13.1; no longer U3.10 (P06)
- net BTN_LOCK: no longer U3.13 (P10)
- net BTN_S1: no longer U3.14 (P11)
- net BTN_S2: no longer U3.15 (P12)
- net GND: now also C13.2, C5.2, D6.1 (A1), D7.1 (A1), D8.1 (A1), D9.1 (A1), J10.2, J10.3; no longer J2.5
- net HALL_LBUMP: now also U3.6 (P02); no longer U3.8 (P04)
- net HALL_LIFT: now also U3.9 (P05); no longer U3.6 (P02)
- net HALL_LIFTX: now also U3.5 (P01); no longer U3.7 (P03)
- net HALL_RBUMP: now also U3.8 (P04); no longer U3.9 (P05)
- net LCD_BACKLIGHT: no longer U4.33 (SPICLK/GPIO30)
- net LED_CHARGE: now also U4.11 (GPIO6/ADC1_CH5); no longer U4.9 (GPIO4/ADC1_CH3)
- net LED_GN: now also U4.52 (GPIO46); no longer U4.34 (SPIQ/GPIO31)
- net LED_LOCK: no longer U4.32 (SPICS0/GPIO29)
- net LED_RD: now also U4.27 (GPIO21); no longer U4.35 (SPID/GPIO32)
- net LED_S2: no longer U4.31 (SPIWP/GPIO28)
- net RAIN: now also U4.19 (GPIO14/ADC2_CH3); no longer U4.22 (GPIO16/ADC2_CH5/XTAL_32K_N)
- net STOP_1: now also U3.7 (P03); no longer U3.4 (P00)
- net STOP_2: now also U3.4 (P00); no longer U3.5 (P01)
- net USB_D+: now also D7.2 (A2)
- net USB_D-: now also D6.2 (A2)
- net at C8.1, L1.1: now also R14.1, R15.1; no longer ANT1.1
- net LED_44HR: now reaches U4.10 (GPIO5/ADC1_CH4)
- net LED_14HR: now reaches U4.12 (GPIO7/ADC1_CH6)
- net LED_24HR: now reaches U4.13 (GPIO8/ADC1_CH7)
- net LED_34HR: now reaches U4.14 (GPIO9/ADC1_CH8)
- net RESET: now reaches C6.1, R7.1, S1.C, S1.D, U4.4 (CHIP_PU/RESET)
- net RESET: now also J2.10
- net at D1.2 (A), J1.1 (VBUS): now also D8.2 (A2)
- net BTN_4H/R4 renamed BTN_44HR
- net JTAG_TCK-SWCLK renamed JTAG_TCK
- net JTAG_TDO-SWD renamed JTAG_TDO
- net JTAG_TMS-SWDIO renamed JTAG_TMS
- net LED_6H/LCD renamed LED_S1
- net LED_CONN_ADS7843-DIN renamed LED_BAT
- net LED_LIFTED_ADS7843_CS renamed LED_LIFTED
- net LED_S1/ADS7843_BUSY: no longer names the net of U4.30 (SPIHD/GPIO27)
- net Shell Stop 1 renamed SHELL_STOP_2
- net Shell Stop 2: no longer names the net of U3.20 (P17)
- new net: ANT1.1, R14.2
- new net: J10.1, R15.2
- new net: D5.2 (A), D9.2 (A2), J2.5
- new net BTN_14HR: U3.13 (P10)
- new net BTN_24HR: U3.14 (P11)
- new net BTN_34HR: U3.15 (P12)
- new net LED_CONN: U4.9 (GPIO4/ADC1_CH3)
- new net SHELL_STOP_1: U3.10 (P06)
- no-connect marks 36 -> 13
Other:
- added sheet Mower Connectors (MowerConnectors.kicad_sch)
- note added: "(Boot Mode)"
- note added: "(Ext. JTAG)"
- note added: "(Weak Pull-Down)"
- note added: "ESP32-S3 Design Guidelines: - Layer 1 (TOP): Signal traces and components. - Layer 2 (GND): No signal traces here to ensure a complete GND plane. - Layer 3 (POWER): GND plane should be applied to better isolate the RF and crystal. Route power traces and a few signal traces on this layer, provided that there is a complete GND plane under the RF and crystal. - Layer 4 (BOTTOM): Route a few signal t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"
- note added: "ROM_MSG_PRNT (Weak Pull-Down)"
- note added: "TODO: - C9 reference value is 1.2-1.8pF - L2 Reference value is 2.4-3.0nH - C8 Reference value is 1.8-1.2pF - UART0-2 are running? Also RXDX/TXDX? - WiFi coverage is acceptable? - Rain?"
- note added: "VDD_SPI (Weak Pull-Down = 3.3V)"
- note removed: "BTN_ANY"
- note removed: "Either use YF-Rev4-A/B or YF-Rev6-A/B connector pair. Adapter get get plugged to the matching CoverUI- A or B side. Other side get plugged either to YF-Mainboard, or remains free and get connected via "OM UI Board" plug to an OpenMower-Mainboard."
- note removed: "If used should become a LED"
- note removed: "JP3.06?"
- note removed: "VDD_SPI Voltage Control"
- moved on the sheet: ANT1, C1, C10, C11, C12, C3, C6, C8, C9, D1, D2, D3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

Commit message: Add HW comment
Other:
- note added: "TODO: - C9 reference value is 1.2-1.8pF - L2 Reference value is 2.4-3.0nH - C8 Reference value is 1.8-1.2pF - UART0-2 are running? Also RXDX/TXDX? - WiFi coverage is acceptable? - Rain? - Chrystal is more sensitive thane before!! Is v0.2 chrystal the same than v0.1? Measure C's and check routing!"
- note removed: "TODO: - C9 reference value is 1.2-1.8pF - L2 Reference value is 2.4-3.0nH - C8 Reference value is 1.8-1.2pF - UART0-2 are running? Also RXDX/TXDX? - WiFi coverage is acceptable? - Rain?"
Changed lines of the file:
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@@
 		)
 	)
-	(text "TODO:\n- C9 reference value is 1.2-1.8pF\n- L2 Reference value is 2.4-3.0nH\n- C8 Reference value is 1.8-1.2pF\n\n- UART0-2 are running? Also RXDX/TXDX?\n- WiFi coverage is acceptable?\n- Rain?"
+	(text "TODO:\n- C9 reference value is 1.2-1.8pF\n- L2 Reference value is 2.4-3.0nH\n- C8 Reference value is 1.8-1.2pF\n\n- UART0-2 are running? Also RXDX/TXDX?\n- WiFi coverage is acceptable?\n- Rain?\n\n- Chrystal is more sensitive thane before!!\n  Is v0.2 chrystal the same than v0.1?\n  Measure C's and check routing!"
 		(exclude_from_sim no)
 		(at 89.662 -7.874 0)
 		(effects
 			(font
+				(face "Bitstream Vera Sans Mono")
 				(size 1.27 1.27)
 			)

Commit message: Prepared HW v0.3
Parts:
- removed GPIO33, GPIO48: TestPoint, TestPoint:TestPoint_Pad_1.0x1.0mm, symbol Connector:TestPoint
- removed J10: IPEX/U.FL, libs:IPEX-SMD_BWIPX-1-001E, symbol 20279-001E-03:20279-001E-03
- removed R14, R15: 0, Resistor_SMD:R_0402_1005Metric, symbol Device:R
- added BOOT-MSG/GPIO46, BOOT/GPIO0, GPIO21: TestPoint, TestPoint:TestPoint_Pad_1.0x1.0mm, symbol Connector:TestPoint
- added J10: MM8130-2600RA2, libs:MURATA_MM8130-2600RA2, symbol MM8130-2600RA2:MM8130-2600RA2
- C8: now not fitted
Connections:
- net BTN_PLAY: now also U3.20 (P17); no longer U4.5 (GPIO0/BOOT)
- net GND: now also J10.GND1 (GND), J10.GND2 (GND__1), J10.GND3 (GND__2), J10.GND4 (GND__3)
- net LED_GN: now also BOOT-MSG/GPIO46.1
- net LED_RD: now also U4.51 (GPIO45); no longer U4.27 (GPIO21)
- net at C8.1, L1.1: now also J10.IN
- net at ANT1.1: now also J10.OUT
- net BTN_ANY: now reaches U4.36 (SPICLK_N/GPIO48)
- net RAIN_OEM: now reaches U4.38 (GPIO33)
- net RAIN renamed RAIN_SENSOR
- new net: GPIO21.1, U4.27 (GPIO21)
- new net: BOOT/GPIO0.1, U4.5 (GPIO0/BOOT)
- no-connect marks 13 -> 11
Other:
- sheet Mower Connectors ports: added BTN_ANY, RAIN_OEM; removed none
- note added: "(Floating)"
- note added: "ESP32-S3 Design Remarks: - GND plane under RF and crystal. - The width of the main power traces should be no less than 25 mil (0,635). The width of VDD3P3 power traces should be no less than 20 mil (0,508mm). The recommended width of other power traces is 10 mil (0,254mm)"
- note added: "TODO: - C9 reference value is 1.2-1.8pF - L2 Reference value is 2.4-3.0nH - C8 Reference value is 1.8-1.2pF - WiFi coverage is acceptable? - Rain? - Chrystal is more sensitive thane before!! Is v0.2 chrystal the same than v0.1? Measure C's and check routing!"
- note removed: "(Boot Mode)"
- note removed: "ESP32-S3 Design Guidelines: - Layer 1 (TOP): Signal traces and components. - Layer 2 (GND): No signal traces here to ensure a complete GND plane. - Layer 3 (POWER): GND plane should be applied to better isolate the RF and crystal. Route power traces and a few signal traces on this layer, provided that there is a complete GND plane under the RF and crystal. - Layer 4 (BOTTOM): Route a few signal t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"
- note removed: "TODO: - C9 reference value is 1.2-1.8pF - L2 Reference value is 2.4-3.0nH - C8 Reference value is 1.8-1.2pF - UART0-2 are running? Also RXDX/TXDX? - WiFi coverage is acceptable? - Rain? - Chrystal is more sensitive thane before!! Is v0.2 chrystal the same than v0.1? Measure C's and check routing!"
- moved on the sheet: ANT1, C9, GPIO47, L1
